File: Relay.sch (KiCad schematic (older format))
At the start: 10 parts

Commit message: arduino module / hooking things up
Connections:
- net labels added: RELAY+, RELAY-, RELAY_COM, RELAY_NC, RELAY_NO
- net labels removed: COM, DIN+, DIN-, NC, NO
Changed lines of the file:
@@
 $EndDescr
 Text HLabel 2550 3400 0    60   Input ~ 0
-DIN+
+RELAY+
 Text HLabel 2550 3750 0    60   Input ~ 0
-DIN-
+RELAY-
 Text HLabel 9050 2900 2    60   BiDi ~ 0
-NC
+RELAY_NC
 Text HLabel 9050 3100 2    60   BiDi ~ 0
-NO
+RELAY_NO
 $Comp
 L PHTRANS U?
@@
 $EndComp
 Text HLabel 9050 2550 2    60   BiDi ~ 0
-COM
+RELAY_COM
 $Comp
 L R R?

Commit message: associating and placing relay module
Parts:
- removed U?: PHTRANS, ~, symbol PHTRANS
- added R6: 0, ~, symbol R
- added U1: OPTO LTV-816S, symbol OPTO-TRANSISTOR4
- D1: renamed from D?; value LED -> LED LG Q971-KN-1; footprint ~ -> 0603; Distributor (none) -> DigiKey; Distributor Link (none) -> http://www.digikey.com/product-detail/en/LG%20Q971-KN-1/475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; Distributor Part Number (none) -> 475-1409-1-ND; MFG Name (none) -> OSRAM Opto Semiconductors Inc; MFG Part Number (none) -> LG Q971-KN-1
- D2: renamed from D?; value DIODE -> SCHOTTKY B130-13-F; Distributor (none) -> DigiKey; Distributor Link (none) -> http://www.digikey.com/product-detail/en/B130-13-F/B130-FDI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; Distributor Part Number (none) -> B130-FDICT-ND; MFG Name (none) -> Diodes Incorporated; MFG Part Number (none) -> B130-13-F
- K1: renamed from K?; Distributor (none) -> DigiKey; Distributor Link (none) -> http://www.digikey.com/product-detail/en/1461069-5/PB1321-N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; Distributor Part Number (none) -> PB1321-ND; MFG Name (none) -> TE Connectivity; MFG Part Number (none) -> 1461069-5
- Q1: renamed from Q?; value NPN -> MMBT3904-7-F; Distributor (none) -> DigiKey; Distributor Link (none) -> http://www.digikey.com/product-detail/en/MMBT3904-7-F/MMBT3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; Distributor Part Number (none) -> MMBT3904-FDICT-ND; MFG Name (none) -> Diodes Incorporated; MFG Part Number (none) -> MMBT3904-7-F
- R1: renamed from R?; value R -> 500
- R2: renamed from R?; value R -> 200
- R3: renamed from R?; value R -> 100
- R4, R5: renamed from R?; value R -> 0
Connections:
- wire segments 34 -> 30
Other:
- moved on the sheet: R1, R4
