File: Power.sch (KiCad schematic (older format))
At the start: 0 parts

Commit message: Power circuit
Parts:
- added C? (x2): C, ~, symbol C
- added F? (x4): FUSE, ~, symbol FUSE
- added L? (x2): INDUCTOR, ~, symbol INDUCTOR
- added P?: CONN_12X2, symbol CONN_12X2
- added R?: R, ~, symbol R
- added SW?: SWITCH_INV, ~, symbol SWITCH_INV
Connections:
- new net: F?.1, P?.1 (P1), P?.2 (P2)
- new net: F?.1, P?.10 (P10)
- new net: F?.1, P?.14 (P14)
- new net: P?.16 (P16), SW?.2
- new net: F?.1, P?.4 (P4), P?.6 (P6)
- new net: R?.1, SW?.1
- new net +12P: F?.2, L?.1
- new net +12V: C?.1, L?.2
- new net +3.3V: F?.2, R?.2
- new net +5V: F?.2
- new net -12P: F?.2, L?.1
- new net -12V: C?.2, L?.2
- new net GND: C?.1, C?.2, P?.3 (P3), P?.5 (P5), SW?.3
Other:
- note added: "Filtering"

Commit message: currentfan revisited
Parts:
- removed F? (x4): FUSE, ~, symbol FUSE
- added TH? (x4): THERMISTOR, ~, symbol THERMISTOR
Connections:
- net +12P: now also TH?.2
- net +3.3V: now also TH?.2
- net +5V: now also TH?.2
- net -12P: now also TH?.2
- net at P?.1 (P1), P?.2 (P2): now also TH?.1
- net +12C: now reaches P?.10 (P10)
- net +12C: now also TH?.1
- net at P?.14 (P14): now also TH?.1
- net at P?.4 (P4), P?.6 (P6): now also TH?.1
Changed lines of the file:
@@
 $Descr A4 11693 8268
 encoding utf-8
-Sheet 4 9
+Sheet 3 9
 Title ""
-Date "7 feb 2014"
+Date "10 feb 2014"
 Rev ""
 Comp ""
@@
 $EndComp
 Wire Wire Line
-	1950 1650 1700 1650
-Wire Wire Line
-	1700 1650 1000 1650
+	1000 1650 1950 1650
 Wire Wire Line
 	1000 1650 1000 1900
-$Comp
-L FUSE F?
-U 1 1 52F3AA3C
-P 3350 1550
-F 0 "F?" H 3450 1600 40  0000 C CNN
-F 1 "FUSE" H 3250 1500 40  0000 C CNN
-F 2 "~" H 3350 1550 60  0000 C CNN
-F 3 "~" H 3350 1550 60  0000 C CNN
-	1    3350 1550
-	1    0    0    -1
-$EndComp
-$Comp
-L FUSE F?
-U 1 1 52F3AA49
-P 3850 1850
-F 0 "F?" H 3950 1900 40  0000 C CNN
-F 1 "FUSE" H 3750 1800 40  0000 C CNN
-F 2 "~" H 3850 1850 60  0000 C CNN
-F 3 "~" H 3850 1850 60  0000 C CNN
-	1    3850 1850
-	1    0    0    -1
-$EndComp
-$Comp
-L FUSE F?
-U 1 1 52F3AA4F
-P 4350 2150
-F 0 "F?" H 4450 2200 40  0000 C CNN
-F 1 "FUSE" H 4250 2100 40  0000 C CNN
-F 2 "~" H 4350 2150 60  0000 C CNN
-F 3 "~" H 4350 2150 60  0000 C CNN
-	1    4350 2150
-	1    0    0    -1
-$EndComp
-$Comp
-L FUSE F?
-U 1 1 52F3AA55
-P 4850 2450
-F 0 "F?" H 4950 2500 40  0000 C CNN
-F 1 "FUSE" H 4750 2400 40  0000 C CNN
-F 2 "~" H 4850 2450 60  0000 C CNN
-F 3 "~" H 4850 2450 60  0000 C CNN
-	1    4850 2450
-	1    0    0    -1
-$EndComp
 Wire Wire Line
 	2750 1750 3100 1750
@@
 	2750 1650 3100 1650
 Wire Wire Line
-	2750 1550 2850 1550
-Wire Wire Line
-	2850 1550 3100 1550
-Wire Wire Line
-	3100 1650 3100 1750
-Wire Wire Line
-	3100 1750 3100 1850
+	2750 1550 3100 1550
+Wire Wire Line
+	3100 1650 3100 1850
 Wire Wire Line
 	3100 1850 3600 1850
@@
 	7600 1550 7750 1550
 Wire Wire Line
-	8350 1550 8550 1550
-Wire Wire Line
-	8550 1550 9000 1550
+	8350 1550 9000 1550
 Wire Wire Line
 	8550 1550 8550 1600
 Wire Wire Line
-	8550 2000 8550 2100
-Wire Wire Line
-	8550 2100 8550 2150
+	8550 2000 8550 2150
 Wire Wire Line
 	8550 2550 8550 2600
 Wire Wire Line
-	8350 2600 8550 2600
-Wire Wire Line
-	8550 2600 9000 2600
+	8350 2600 9000 2600
 Wire Wire Line
 	7750 2600 7600 2600
@@
 Text Notes 8200 3050 0    60   ~ 0
 Filtering
+Wire Wire Line
+	2950 1950 2950 1100
+Connection ~ 2950 1950
+$Comp
+L +12C #PWR?
+U 1 1 52F8F8DF
+P 2950 1100
+F 0 "#PWR?" H 3000 1150 60  0001 C CNN
+F 1 "+12C" H 2950 1100 60  0001 C CNN
+F 2 "" H 2950 1100 60  0000 C CNN
+F 3 "" H 2950 1100 60  0001 C CNN
+F 4 "#PWR" H 2950 1070 30  0001 C CNN "Reference"
+F 5 "+12C" H 2950 1210 40  0000 C CNN "Value"
+F 6 "" H 2950 1100 60  0000 C CNN "Datasheet"
+	1    2950 1100
+	1    0    0    -1
+$EndComp
+$Comp
+L THERMISTOR TH?
+U 1 1 52F8FA4B
+P 3350 1550
+F 0 "TH?" H 3400 1600 60  0001 C CNN
+F 1 "THERMISTOR" H 3350 1550 60  0001 C CNN
+F 2 "~" H 3350 1550 60  0000 C CNN
+F 3 "" H 3350 1550 60  0001 C CNN
+F 4 "TH" V 3450 1600 50  0000 C CNN "Reference"
+F 5 "THERMISTOR" V 3250 1550 50  0000 C CNN "Value"
+F 6 "~" H 3350 1550 60  0000 C CNN "Datasheet"
+	1    3350 1550
+	0    -1   -1   0
+$EndComp
+$Comp
+L THERMISTOR TH?
+U 1 1 52F8FA72
+P 3850 1850
+F 0 "TH?" H 3900 1900 60  0001 C CNN
+F 1 "THERMISTOR" H 3850 1850 60  0001 C CNN
+F 2 "~" H 3850 1850 60  0000 C CNN
+F 3 "" H 3850 1850 60  0001 C CNN
+F 4 "TH" V 3950 1900 50  0000 C CNN "Reference"
+F 5 "THERMISTOR" V 3750 1850 50  0000 C CNN "Value"
+F 6 "~" H 3850 1850 60  0000 C CNN "Datasheet"
+	1    3850 1850
+	0    -1   -1   0
+$EndComp
+$Comp
+L THERMISTOR TH?
+U 1 1 52F8FA7B
+P 4350 2150
+F 0 "TH?" H 4400 2200 60  0001 C CNN
+F 1 "THERMISTOR" H 4350 2150 60  0001 C CNN
+F 2 "~" H 4350 2150 60  0000 C CNN
+F 3 "" H 4350 2150 60  0001 C CNN
+F 4 "TH" V 4450 2200 50  0000 C CNN "Reference"
+F 5 "THERMISTOR" V 4250 2150 50  0000 C CNN "Value"
+F 6 "~" H 4350 2150 60  0000 C CNN "Datasheet"
+	1    4350 2150
+	0    -1   -1   0
+$EndComp
+$Comp
+L THERMISTOR TH?
+U 1 1 52F8FA84
+P 4850 2450
+F 0 "TH?" H 4900 2500 60  0001 C CNN
+F 1 "THERMISTOR" H 4850 2450 60  0001 C CNN
+F 2 "~" H 4850 2450 60  0000 C CNN
+F 3 "" H 4850 2450 60  0001 C CNN
+F 4 "TH" V 4950 2500 50  0000 C CNN "Reference"
+F 5 "THERMISTOR" V 4750 2450 50  0000 C CNN "Value"
+F 6 "~" H 4850 2450 60  0000 C CNN "Datasheet"
+	1    4850 2450
+	0    -1   -1   0
+$EndComp
 $EndSCHEMATC
