File: $Thermalcouple.sch (KiCad schematic (older format))
At the start: 20 parts, among them P2 CONN_3X2, P3 CONN_2, U3 MCP3901, U4 LMT84, U5 OPA4170

Commit message: associating-and-placing-the-thermocouple-module
Parts:
- added R41, R42: 0, ~, symbol R
Connections:
- net AGND: now also R41.1, R42.1; no longer C7.2, U3.5 (CH0-), U3.7 (CH1-)
- new net CH0-: C7.2, R42.2, U3.5 (CH0-)
- new net CH1-: R41.2, U3.7 (CH1-)
Changed lines of the file:
@@
 L AGND #PWR029
 U 1 1 52F0F60A
-P 5650 4150
-F 0 "#PWR029" H 5650 4150 40  0001 C CNN
-F 1 "AGND" H 5650 4080 50  0000 C CNN
-F 2 "" H 5650 4150 60  0000 C CNN
-F 3 "" H 5650 4150 60  0000 C CNN
-	1    5650 4150
-	1    0    0    -1
-$EndComp
-Wire Wire Line
-	5650 3950 5950 3950
-Wire Wire Line
-	5650 3200 5650 4150
-Connection ~ 5650 3950
+P 5550 4150
+F 0 "#PWR029" H 5550 4150 40  0001 C CNN
+F 1 "AGND" H 5550 4080 50  0000 C CNN
+F 2 "" H 5550 4150 60  0000 C CNN
+F 3 "" H 5550 4150 60  0000 C CNN
+	1    5550 4150
+	1    0    0    -1
+$EndComp
+Wire Wire Line
+	5550 3950 5950 3950
 $Comp
 L AGND #PWR030
@@
 Connection ~ 5650 3000
 Wire Wire Line
-	5650 3200 4650 3200
+	5550 3200 4650 3200
 Wire Wire Line
 	1100 2700 2000 2700
@@
 Connection ~ 5900 3000
 Wire Wire Line
-	5900 3450 5900 3550
-Wire Wire Line
-	5900 3550 5650 3550
-Connection ~ 5650 3550
+	5550 3450 5900 3450
 $Comp
 L R R37
@@
 Wire Wire Line
 	4750 6200 6300 6200
-Wire Wire Line
-	4750 4000 4750 6350
 Wire Wire Line
 	5900 6100 5900 6200
@@
 Text Label 4700 4000 0    60   ~ 0
 CH1-
+$Comp
+L R R42
+U 1 1 530A6D0B
+P 5550 3700
+F 0 "R42" V 5630 3700 40  0000 C CNN
+F 1 "0" V 5557 3701 40  0000 C CNN
+F 2 "~" V 5480 3700 30  0000 C CNN
+F 3 "~" H 5550 3700 30  0000 C CNN
+	1    5550 3700
+	-1   0    0    1
+$EndComp
+Wire Wire Line
+	5550 3450 5550 3200
+$Comp
+L R R41
+U 1 1 530A6E02
+P 4750 5250
+F 0 "R41" V 4830 5250 40  0000 C CNN
+F 1 "0" V 4757 5251 40  0000 C CNN
+F 2 "~" V 4680 5250 30  0000 C CNN
+F 3 "~" H 4750 5250 30  0000 C CNN
+	1    4750 5250
+	-1   0    0    1
+$EndComp
+Wire Wire Line
+	4750 4000 4750 5000
+Wire Wire Line
+	4750 5500 4750 6350
+Wire Wire Line
+	5550 3950 5550 4150
 $EndSCHEMATC
