File: BenchBuddy.kicad_pcb (KiCad board)
At the start: 4 copper layers, 166.4 x 64.8 mm, 12 parts, among them K1 RELAY_SPDT 1461069-5, Q1 MMBT3904-7-F, U1 OPTO LTV-816S, U8 MCP4922-E/ST

Commit message: associating-and-placing-the-thermocouple-module
Parts:
- removed U8: MCP4922-E/ST, TSSOP14
- added C10: C, SM0805, F.Cu at (240.7, 156.2)
- added C11: C, SM0805, B.Cu at (283.2, 171.4)
- added C12: C, SM0805, B.Cu at (243.2, 167.6)
- added C7: C, SM0805, B.Cu at (238.1, 167.0)
- added C8: C, SM0805, B.Cu at (227.3, 168.9)
- added C9: C, SM0805, B.Cu at (227.3, 167.0)
- added P2: CONN_3X2, pin_array_3x2, F.Cu at (240.0, 147.3)
- added P3: CONN_2, PIN_ARRAY_2X1, F.Cu at (219.7, 163.8)
- added R10: R, SM1206, B.Cu at (240.7, 168.9)
- added R11: R, SM1206, B.Cu at (243.8, 159.4)
- added R12: R, SM1206, B.Cu at (237.5, 159.4)
- added R13: R, SM1206, B.Cu at (247.0, 159.4)
- added R14: R, SM0805, B.Cu at (237.5, 152.4)
- added R15: R, SM1206, B.Cu at (240.7, 159.4)
- added R37: R, SM0805, B.Cu at (240.0, 152.4)
- added R38: R, SM0805, B.Cu at (242.6, 152.4)
- added R41: 0, SM0805, B.Cu at (236.2, 170.8)
- added R42: 0, SM0805, B.Cu at (238.1, 170.8)
- added R9: R, SM1206, B.Cu at (238.8, 163.8)
- added U3: MCP3901, SSOP20, F.Cu at (227.3, 165.7)
- added U4: LMT84, SOT353, F.Cu at (283.2, 168.9)
- added U5: OPA4170, SO14E, F.Cu at (241.9, 161.3)
- K1: value RELAY_SPDT 1461069-5 -> RELAY_SPDT
Other:
- board size 166.4 x 64.8 mm -> 165.1 x 63.5 mm

Commit message: associating-and-placing-the-terminal-atx-blocks
Parts:
- added K2: 3 Pin Terminal Block, 3pinTB, F.Cu at (284.5, 125.7)
- added P1: 24 Pin Minifit Jr, 24pin-ATX, F.Cu at (137.2, 120.7)
- added P4: 12 Pin Terminal Block, 12pinTB, F.Cu at (285.1, 172.1)
- moved C11 7.01 mm to (276.2, 172.1)
- moved U4 6.98 mm to (276.2, 168.9)
Connections:
- K1 pad 1: (no net) -> /Relay/RELAY_COM
- K1 pad 3: (no net) -> /TerminalBlock/RELAY_NC
- K1 pad 4: (no net) -> /Relay/RELAY_NC
- U5 pad 10: (no net) -> /Thermalcouple/TC IN +

Commit message: associating-and-placing-arduino-module
Parts:
- added R23: 0, SM0805, F.Cu at (188.6, 164.5)
- added R24: 0, SM0805, F.Cu at (191.1, 164.5)
- added R25: 0, SM0805, F.Cu at (193.7, 164.5)
- added R26: 0, SM0805, F.Cu at (196.2, 164.5)
- added R27: 0, SM0805, F.Cu at (198.8, 164.5)
- added R28: 0, SM0805, F.Cu at (192.4, 124.5)
- added R29: 0, SM0805, F.Cu at (194.9, 124.5)
- added R30: 0, SM0805, F.Cu at (198.8, 124.5)
- added R31: 0, SM0805, F.Cu at (201.3, 124.5)
- added R32: 0, SM0805, F.Cu at (203.8, 124.5)
- added R33: 0, SM0805, F.Cu at (206.4, 124.5)
- added R34: 0, SM0805, F.Cu at (208.9, 124.5)
- added R35: 0, SM0805, F.Cu at (211.5, 164.5)
- added R36: 0, SM0805, F.Cu at (208.9, 164.5)
- added R39: 0, SM0805, F.Cu at (214.0, 124.5)
- added R40: 0, SM0805, F.Cu at (216.5, 124.5)
- added U10: ARDUINOPINS, ArduinoUnoR3, F.Cu at (153.0, 170.8)
- moved P3 11.2 mm to (227.3, 172.1), turned to 180 degrees

Commit message: fan module
Parts:
- added C13: C, SM0805, F.Cu at (243.2, 173.4)
- added C14: C, SM0805, B.Cu at (255.9, 165.1)
- added D5: B130-13-F, SMA, F.Cu at (266.1, 170.8)
- added Q2: DMN65D8L-7, SOT23GDS, F.Cu at (238.1, 170.8)
- added Q3: AOD476, DPAK2, F.Cu at (255.9, 164.5)
- added Q4: AOD476, DPAK2, F.Cu at (264.8, 165.1)
- added R21: R, SM0805, F.Cu at (234.3, 168.3)
- added R22: 1, SM1206, F.Cu at (243.8, 169.5)
- added TH5: PTC 500mA, SM1812, B.Cu at (264.8, 165.1)
- added U8: MCP4801, SO8E, F.Cu at (228.0, 170.2)
- R23, R24, R25, R26, R27, R28, R29, R30, R31, R32, R33, R34, R35, R36, R39, R4, R40, R41, R42, R5, R6: footprint SM0805 -> S_Jumper_SM0805
- moved C8 17.2 mm to (226.7, 151.8)
- moved P3 17.2 mm to (226.7, 154.9)
- moved C9 17.2 mm to (226.7, 149.9)
- moved U3 10.8 mm to (227.3, 154.9)
- moved C10 7.62 mm to (240.7, 148.6)
- moved C7 7.62 mm to (238.1, 159.4)
- moved P2 7.62 mm to (240.0, 139.7)
- moved R10 7.62 mm to (240.7, 161.3)
- moved R11 7.62 mm to (243.8, 151.8)
- moved R12 7.62 mm to (237.5, 151.8)
- moved R14 7.62 mm to (237.5, 144.8)
- moved R15 7.62 mm to (240.7, 151.8)
- moved R37 7.62 mm to (240.0, 144.8)
- moved R38 7.62 mm to (242.6, 144.8)
- moved R41 7.62 mm to (236.2, 163.2)
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Connections:
- net /Arduino/ADC_CS_N renamed /Arduino/~ADC_CS
- U10 pad 13: (no net) -> N-0000045
- U10 pad 14: (no net) -> N-0000056
